File: pcb/controller/controller.kicad_pcb (KiCad board)
At the start: 2 copper layers, 90 x 65 mm, 40 parts, among them J1 Barrel_Jack, J2 AVR-ISP-6, U1 ATmega328P-A, Y1 Crystal_GND24

Commit message: Controller PCB Diagnostic Header
This adds a diagnostic header that I'll be able to put a jumper on to
turn on diagnostic mode--which will be used to calibrate the
potentiometer inputs.  In addition to adding this to the PCB layout, I
rearranged a few components and cleaned up some traces.
Parts:
- added JDIAG1: Conn_01x03_Male, Connector_PinHeader_2.54mm:PinHeader_1x03_P2.54mm_Vertical, F.Cu at (153.0, 73.0)
- moved C2 27.0 mm to (178.1, 89.0), turned to 180 degrees
- moved C1 23.4 mm to (178.1, 94.0), turned to 180 degrees
- moved C4 5.00 mm to (152.0, 89.0), turned to 90 degrees
- moved C3 4.24 mm to (158.0, 87.0), turned to 180 degrees
- moved R1 2.96 mm to (146.4, 77.5)
Connections:
- U1 pad 1: unconnected-(U1-Pad1) -> Net-(U1-Pad1)
Routing:
- net Net-(U1-Pad1): track 0.00 -> 25.1 mm, vias 0 -> 1
- net GND: track 50.9 -> 41.6 mm, vias 12 -> 8
- net Net-(C3-Pad2): track 19.1 -> 12.7 mm, vias 2 -> 0
- net Net-(D1-Pad1): track 5.82 -> 8.97 mm
- net Net-(C4-Pad2): track 16.4 -> 17.9 mm
