File: pcb/digit/digit.kicad_sch (KiCad schematic)
At the start: 23 parts

Commit message: Added Separator PCB And Build Files
This adds a simple PCB with 2 WS2812B LEDs for the center separator.
I also generated gerber, BOM and pick and place files for all the
boards and updated the part numbers for the WS2812B LEDs to the new
version that JLCPCB carries.
Parts:
- D1: LCSC C2846931 -> C2874885
- D10, D11, D12, D13, D14, D15, D16, D17, D18, D19, D2, D20, D21, D3, D4, D5, D6, D7, D8, D9: LCSC (none) -> C2874885
Changed lines of the file:
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@@
       (effects (font (size 1.27 1.27)) (justify left top) hide)
+    )
+    (property "LCSC" "C2874885" (id 4) (at 219.71 63.5 0)
+      (effects (font (size 1.27 1.27)) hide)
     )
     (pin "1")
@@
       (effects (font (size 1.27 1.27)) (justify left top) hide)
     )
+    (property "LCSC" "C2874885" (id 4) (at 113.03 63.5 0)
+      (effects (font (size 1.27 1.27)) hide)
+    )
     (pin "1")
     (pin "2")
@@
       (effects (font (size 1.27 1.27)) (justify left top) hide)
     )
+    (property "LCSC" "C2874885" (id 4) (at 67.31 91.44 0)
+      (effects (font (size 1.27 1.27)) hide)
+    )
     (pin "1")
     (pin "2")
@@
       (effects (font (size 1.27 1.27)) (justify left top) hide)
     )
+    (property "LCSC" "C2874885" (id 4) (at 82.55 63.5 0)
+      (effects (font (size 1.27 1.27)) hide)
+    )
     (pin "1")
     (pin "2")
@@
       (effects (font (size 1.27 1.27)) (justify left top) hide)
     )
+    (property "LCSC" "C2874885" (id 4) (at 143.51 63.5 0)
+      (effects (font (size 1.27 1.27)) hide)
+    )
     (pin "1")
     (pin "2")
@@
       (effects (font (size 1.27 1.27)) (justify left top) hide)
     )
+    (property "LCSC" "C2874885" (id 4) (at 234.95 63.5 0)
+      (effects (font (size 1.27 1.27)) hide)
+    )
     (pin "1")
     (pin "2")
@@
       (effects (font (size 1.27 1.27)) (justify left top) hide)
     )
+    (property "LCSC" "C2874885" (id 4) (at 52.07 91.44 0)
+      (effects (font (size 1.27 1.27)) hide)
+    )
     (pin "1")
     (pin "2")
@@
       (effects (font (size 1.27 1.27)) (justify left top) hide)
     )
+    (property "LCSC" "C2874885" (id 4) (at 204.47 63.5 0)
+      (effects (font (size 1.27 1.27)) hide)
+    )
     (pin "1")
     (pin "2")
@@
       (effects (font (size 1.27 1.27)) (justify left top) hide)
     )
+    (property "LCSC" "C2874885" (id 4) (at 97.79 63.5 0)
+      (effects (font (size 1.27 1.27)) hide)
+    )
     (pin "1")
     (pin "2")
@@
       (effects (font (size 1.27 1.27)) (justify left top) hide)
     )
+    (property "LCSC" "C2874885" (id 4) (at 113.03 91.44 0)
+      (effects (font (size 1.27 1.27)) hide)
+    )
     (pin "1")
     (pin "2")
@@
       (effects (font (size 1.27 1.27)) (justify left top) hide)
     )
+    (property "LCSC" "C2874885" (id 4) (at 250.19 63.5 0)
+      (effects (font (size 1.27 1.27)) hide)
+    )
     (pin "1")
     (pin "2")
@@
       (effects (font (size 1.27 1.27)) (justify left top) hide)
     )
+    (property "LCSC" "C2874885" (id 4) (at 189.23 63.5 0)
+      (effects (font (size 1.27 1.27)) hide)
+    )
     (pin "1")
     (pin "2")
@@
       (effects (font (size 1.27 1.27)) (justify left top) hide)
     )
+    (property "LCSC" "C2874885" (id 4) (at 97.79 91.44 0)
+      (effects (font (size 1.27 1.27)) hide)
+    )
     (pin "1")
     (pin "2")
@@
       (effects (font (size 1.27 1.27)) (justify left top) hide)
     )
+    (property "LCSC" "C2874885" (id 4) (at 173.99 63.5 0)
+      (effects (font (size 1.27 1.27)) hide)
+    )
     (pin "1")
     (pin "2")
@@
       (effects (font (size 1.27 1.27)) (justify left top) hide)
     )
+    (property "LCSC" "C2874885" (id 4) (at 67.31 63.5 0)
+      (effects (font (size 1.27 1.27)) hide)
+    )
     (pin "1")
     (pin "2")
@@
       (effects (font (size 1.27 1.27)) (justify left top) hide)
     )
+    (property "LCSC" "C2874885" (id 4) (at 128.27 91.44 0)
+      (effects (font (size 1.27 1.27)) hide)
+    )
     (pin "1")
     (pin "2")
@@
       (effects (font (size 1.27 1.27)) (justify left top) hide)
     )
+    (property "LCSC" "C2874885" (id 4) (at 143.51 91.44 0)
+      (effects (font (size 1.27 1.27)) hide)
+    )
     (pin "1")
     (pin "2")
@@
       (effects (font (size 1.27 1.27)) (justify left top) hide)
     )
-    (property "LCSC" "C2846931" (id 4) (at 52.07 63.5 0)
+    (property "LCSC" "C2874885" (id 4) (at 52.07 63.5 0)
       (effects (font (size 1.27 1.27)) hide)
     )
@@
       (effects (font (size 1.27 1.27)) (justify left top) hide)
     )
+    (property "LCSC" "C2874885" (id 4) (at 52.07 63.5 0)
+      (effects (font (size 1.27 1.27)) hide)
+    )
     (pin "1")
     (pin "2")
@@
       (effects (font (size 1.27 1.27)) (justify left top) hide)
     )
+    (property "LCSC" "C2874885" (id 4) (at 52.07 63.5 0)
+      (effects (font (size 1.27 1.27)) hide)
+    )
     (pin "1")
     (pin "2")
@@
       (effects (font (size 1.27 1.27)) (justify left top) hide)
     )
-    (pin "1")
+    (property "LCSC" "C2874885" (id 4) (at 52.07 63.5 0)
+      (effects (font (size 1.27 1.27)) hide)
+    )
+    (pin "1")
