File: pcb/digit/digit.kicad_pcb (KiCad board)
At the start: 2 copper layers, 70 x 125 mm, 25 parts

Commit message: PCB Touchup
Two changes in this commit.

1. I rewired the volume potentiometer so that the MOSFET is now the
closest thing to ground.  That way we'll always be sure to have
sufficient gate-source voltage to trigger it when the buzzer is turned
on.

2. I added v1/date indicators to the silk screen layers of all the
PCBs.
Other:
- board text added: "v1 2022-11-12"
Changed lines of the file:
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@@
       (drillshape 0)
       (scaleselection 1)
-      (outputdirectory "bom/")
+      (outputdirectory "gerbers/")
     )
   )
@@
       (xy 126 43)
     ) (layer "Edge.Cuts") (width 0.1) (fill none))
+  (gr_text "v1 2022-11-12" (at 119 45) (layer "B.SilkS")
+    (effects (font (size 1 1) (thickness 0.15)) (justify mirror))
+  )
   (segment (start 83 116) (end 82.45 116.55) (width 1) (layer "F.Cu") (net 1))
   (segment (start 123 124) (end 124.55 122.45) (width 1) (layer "F.Cu") (net 1))
