File: pcb/separator/separator.kicad_pcb (KiCad board)
At the start: 2 copper layers, 14 x 77 mm, 6 parts

Commit message: PCB Touchup
Two changes in this commit.

1. I rewired the volume potentiometer so that the MOSFET is now the
closest thing to ground.  That way we'll always be sure to have
sufficient gate-source voltage to trigger it when the buzzer is turned
on.

2. I added v1/date indicators to the silk screen layers of all the
PCBs.
Other:
- board text added: "2022-11-12"
- board text added: "v1"
Changed lines of the file:
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@@
       (drillshape 0)
       (scaleselection 1)
-      (outputdirectory "bom")
+      (outputdirectory "gerbers/")
     )
   )
@@
       (xy 143 52)
     ) (layer "Edge.Cuts") (width 0.1) (fill none))
+  (gr_text "2022-11-12" (at 143 121) (layer "B.SilkS")
+    (effects (font (size 1 1) (thickness 0.15)) (justify mirror))
+  )
+  (gr_text "v1" (at 143 123) (layer "B.SilkS")
+    (effects (font (size 1 1) (thickness 0.15)) (justify mirror))
+  )
   (segment (start 140.55 111.45) (end 141 111) (width 1) (layer "F.Cu") (net 1))
   (segment (start 140.55 60.45) (end 141 60) (width 1) (layer "F.Cu") (net 1))
